File: acquisition/board/psu.kicad_sch (KiCad schematic)
At the start: 62 parts, among them U25 LTC3374-QFN, U26 LT3042, U27 LT3042, U28 ADR510, U30 LDO1117-12

Commit message: Finished footprint assignment
Parts:
- U25: footprint (none) -> azonenberg_pcb:QFN_38_0.5MM_5x7MM
- U26, U27: footprint (none) -> azonenberg_pcb:DFN_10_0.5MM_3x3MM
- U28: footprint (none) -> azonenberg_pcb:SOT23_3
- U30: footprint (none) -> azonenberg_pcb:SOT223-4
Changed lines of the file:
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@@
   (title_block
     (title "Digitizer board")
-    (date "2022-07-17")
+    (date "2023-01-29")
     (rev "0.1")
     (company "A. Zonenberg")
@@
       (effects (font (size 1.524 1.524)))
     )
-    (property "Footprint" "" (id 2) (at 60.96 189.23 0)
+    (property "Footprint" "azonenberg_pcb:QFN_38_0.5MM_5x7MM" (id 2) (at 60.96 189.23 0)
       (effects (font (size 1.524 1.524)) hide)
     )
@@
       (effects (font (size 1.524 1.524)) (justify left))
     )
-    (property "Footprint" "" (id 2) (at 58.42 27.94 0)
+    (property "Footprint" "azonenberg_pcb:QFN_38_0.5MM_5x7MM" (id 2) (at 58.42 27.94 0)
       (effects (font (size 1.524 1.524)) hide)
     )
@@
       (effects (font (size 1.524 1.524)) (justify left))
     )
-    (property "Footprint" "" (id 2) (at 58.42 110.49 0)
+    (property "Footprint" "azonenberg_pcb:QFN_38_0.5MM_5x7MM" (id 2) (at 58.42 110.49 0)
       (effects (font (size 1.524 1.524)) hide)
     )
@@
       (effects (font (size 1.524 1.524)) (justify left))
     )
-    (property "Footprint" "" (id 2) (at 58.42 77.47 0)
+    (property "Footprint" "azonenberg_pcb:QFN_38_0.5MM_5x7MM" (id 2) (at 58.42 77.47 0)
       (effects (font (size 1.524 1.524)) hide)
     )
@@
       (effects (font (size 1.524 1.524)) (justify left))
     )
-    (property "Footprint" "" (id 2) (at 58.42 60.96 0)
+    (property "Footprint" "azonenberg_pcb:QFN_38_0.5MM_5x7MM" (id 2) (at 58.42 60.96 0)
       (effects (font (size 1.524 1.524)) hide)
     )
@@
       (effects (font (size 1.524 1.524)) (justify left))
     )
-    (property "Footprint" "" (id 2) (at 58.42 44.45 0)
+    (property "Footprint" "azonenberg_pcb:QFN_38_0.5MM_5x7MM" (id 2) (at 58.42 44.45 0)
       (effects (font (size 1.524 1.524)) hide)
     )
@@
       (effects (font (size 1.524 1.524)))
     )
-    (property "Footprint" "" (id 2) (at 168.91 25.4 0)
+    (property "Footprint" "azonenberg_pcb:SOT223-4" (id 2) (at 168.91 25.4 0)
       (effects (font (size 1.524 1.524)) hide)
     )
@@
       (effects (font (size 1.524 1.524)) (justify left))
     )
-    (property "Footprint" "" (id 2) (at 58.42 93.98 0)
+    (property "Footprint" "azonenberg_pcb:QFN_38_0.5MM_5x7MM" (id 2) (at 58.42 93.98 0)
       (effects (font (size 1.524 1.524)) hide)
     )
@@
     (property "Reference" "U28" (id 0) (at 165.1 64.6643 0))
     (property "Value" "ADR510" (id 1) (at 165.1 67.4394 0))
-    (property "Footprint" "" (id 2) (at 157.48 73.66 0)
+    (property "Footprint" "azonenberg_pcb:SOT23_3" (id 2) (at 157.48 73.66 0)
       (effects (font (size 1.27 1.27)) hide)
     )
@@
       (effects (font (size 1.524 1.524)) (justify left))
     )
-    (property "Footprint" "" (id 2) (at 58.42 143.51 0)
+    (property "Footprint" "azonenberg_pcb:QFN_38_0.5MM_5x7MM" (id 2) (at 58.42 143.51 0)
       (effects (font (size 1.524 1.524)) hide)
     )
@@
     (property "Reference" "U26" (id 0) (at 165.735 93.9505 0))
     (property "Value" "LT3042" (id 1) (at 165.735 96.7256 0))
-    (property "Footprint" "" (id 2) (at 157.48 118.11 0)
+    (property "Footprint" "azonenberg_pcb:DFN_10_0.5MM_3x3MM" (id 2) (at 157.48 118.11 0)
       (effects (font (size 1.27 1.27)) hide)
     )
@@
     (property "Reference" "U27" (id 0) (at 165.735 120.6205 0))
     (property "Value" "LT3042" (id 1) (at 165.735 123.3956 0))
-    (property "Footprint" "" (id 2) (at 157.48 144.78 0)
+    (property "Footprint" "azonenberg_pcb:DFN_10_0.5MM_3x3MM" (id 2) (at 157.48 144.78 0)
       (effects (font (size 1.27 1.27)) hide)
     )
@@
       (effects (font (size 1.524 1.524)) (justify left))
     )
-    (property "Footprint" "" (id 2) (at 58.42 127 0)
+    (property "Footprint" "azonenberg_pcb:QFN_38_0.5MM_5x7MM" (id 2) (at 58.42 127 0)
       (effects (font (size 1.524 1.524)) hide)
     )
