File: acquisition/board/adcs.kicad_sch (KiCad schematic)
At the start: 107 parts, among them U1 AD9251, U2 XC7A50T-1FTG256C, U3 AD9251, U4 AD9251, U5 AD9251, U6 ICE40UP5K_QFN48

Commit message: Began layout of clocking subsystem
Connections:
- net ADC2_CS_N: now also U2.H4 (IO_L18N_T2_35); no longer U2.E5 (IO_L13N_T2_MRCC_35)
- net ADC2_OE_N: now also U2.G4 (IO_L16N_T2_35); no longer U2.M12 (IO_L6N_T0_D08_VREF_14)
- net D3_0: now also U2.L2 (IO_L23N_T3_35); no longer U2.E6 (IO_0_35)
- net D3_1: now also U2.K1 (IO_L22P_T3_35); no longer U2.B7 (IO_L1P_T0_AD4P_35)
- net D3_10: now also U2.E1 (IO_L15N_T2_DQS_35); no longer U2.C6 (IO_L5N_T0_AD13N_35)
- net D3_11: now also U2.E2 (IO_L10P_T1_AD15P_35); no longer U2.D6 (IO_L6P_T0_35)
- net D3_12: now also U2.D1 (IO_L10N_T1_AD15N_35); no longer U2.D5 (IO_L6N_T0_VREF_35)
- net D3_13: now also U2.C1 (IO_L9P_T1_DQS_AD7P_35); no longer U2.C3 (IO_L7P_T1_AD6P_35)
- net D3_2: now also U2.K2 (IO_L24N_T3_35); no longer U2.A7 (IO_L1N_T0_AD4N_35)
- net D3_3: now also U2.J1 (IO_L22N_T3_35); no longer U2.B6 (IO_L2P_T0_AD12P_35)
- net D3_4: now also U2.J3 (IO_L21P_T3_DQS_35); no longer U2.B5 (IO_L2N_T0_AD12N_35)
- net D3_5: now also U2.H1 (IO_L20P_T3_35); no longer U2.A5 (IO_L3P_T0_DQS_AD5P_35)
- net D3_6: now also U2.H2 (IO_L20P_T3_35); no longer U2.A4 (IO_L3N_T0_DQS_AD5N_35)
- net D3_7: now also U2.G1 (IO_L17N_T2_35); no longer U2.B4 (IO_L4P_T0_35)
- net D3_8: now also U2.G2 (IO_L17P_T2_35); no longer U2.A3 (IO_L4N_T0_35)
- net D3_9: now also U2.F2 (IO_L15P_T2_DQS_35); no longer U2.C7 (IO_L5P_T0_AD13P_35)
- net D4_0: now also U2.C2 (IO_L7N_T1_AD6N_35); no longer U2.H4 (IO_L18N_T2_35)
- net D4_1: now also U2.B1 (IO_L9N_T1_DQS_AD7N_35); no longer U2.J5 (IO_L19P_T3_35)
- net D4_10: now also U2.H3 (IO_L21P_T3_DQS_35); no longer U2.L2 (IO_L23N_T3_35)
- net D4_11: now also U2.J5 (IO_L19P_T3_35); no longer U2.K3 (IO_L24P_T3_35)
- net D4_12: now also U2.J4 (IO_L19N_T3_VREF_35); no longer U2.K2 (IO_L24N_T3_35)
- net D4_13: now also U2.K3 (IO_L24P_T3_35); no longer U2.K5 (IO_25_35)
- net D4_2: now also U2.A2 (IO_L8N_T1_AD14N_35); no longer U2.J4 (IO_L19N_T3_VREF_35)
- net D4_3: now also U2.B2 (IO_L8P_T1_AD14P_35); no longer U2.H2 (IO_L20P_T3_35)
- net D4_4: now also U2.A3 (IO_L4N_T0_35); no longer U2.H1 (IO_L20P_T3_35)
- net D4_5: now also U2.A4 (IO_L3N_T0_DQS_AD5N_35); no longer U2.J3 (IO_L21P_T3_DQS_35)
- net D4_6: now also U2.B4 (IO_L4P_T0_35); no longer U2.H3 (IO_L21P_T3_DQS_35)
- net D4_7: now also U2.A5 (IO_L3P_T0_DQS_AD5P_35); no longer U2.K1 (IO_L22P_T3_35)
- net D4_8: now also U2.B5 (IO_L2N_T0_AD12N_35); no longer U2.J1 (IO_L22N_T3_35)
- net D4_9: now also U2.A7 (IO_L1N_T0_AD4N_35); no longer U2.L3 (IO_L23P_T3_35)
- net D5_0: now also U2.E5 (IO_L13N_T2_MRCC_35); no longer U2.C2 (IO_L7N_T1_AD6N_35)
- net D5_1: now also U2.B6 (IO_L2P_T0_AD12P_35); no longer U2.B2 (IO_L8P_T1_AD14P_35)
- net D5_10: now also U2.M12 (IO_L6N_T0_D08_VREF_14); no longer U2.G4 (IO_L16N_T2_35)
- net D5_11: now also U2.B7 (IO_L1P_T0_AD4P_35); no longer U2.G2 (IO_L17P_T2_35)
- net D5_12: now also U2.E6 (IO_0_35); no longer U2.G1 (IO_L17N_T2_35)
- net D5_2: now also U2.L3 (IO_L23P_T3_35); no longer U2.A2 (IO_L8N_T1_AD14N_35)
- net D5_3: now also U2.C3 (IO_L7P_T1_AD6P_35); no longer U2.C1 (IO_L9P_T1_DQS_AD7P_35)
- net D5_4: now also U2.K5 (IO_25_35); no longer U2.B1 (IO_L9N_T1_DQS_AD7N_35)
- net D5_5: now also U2.D6 (IO_L6P_T0_35); no longer U2.E2 (IO_L10P_T1_AD15P_35)
- net D5_6: now also U2.D5 (IO_L6N_T0_VREF_35); no longer U2.D1 (IO_L10N_T1_AD15N_35)
- net D5_7: now also U2.C7 (IO_L5P_T0_AD13P_35); no longer U2.F2 (IO_L15P_T2_DQS_35)
- net D5_8: now also U2.C6 (IO_L5N_T0_AD13N_35); no longer U2.E1 (IO_L15N_T2_DQS_35)
Changed lines of the file:
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@@
   (title_block
     (title "Digitizer board")
-    (date "2023-01-31")
+    (date "2023-02-01")
     (rev "0.1")
     (company "A. Zonenberg")
@@
     (effects (font (size 1.27 1.27)) (justify left bottom))
   )
-  (label "D3_10" (at 195.58 172.72 180)
+  (label "D3_10" (at 195.58 223.52 180)
     (effects (font (size 1.27 1.27)) (justify right bottom))
   )
@@
     (effects (font (size 1.27 1.27)) (justify right bottom))
   )
-  (label "D5_1" (at 195.58 185.42 180)
+  (label "D5_1" (at 195.58 154.94 180)
     (effects (font (size 1.27 1.27)) (justify right bottom))
   )
@@
     (effects (font (size 1.27 1.27)) (justify right bottom))
   )
-  (label "D4_9" (at 195.58 261.62 180)
+  (label "D4_9" (at 195.58 152.4 180)
     (effects (font (size 1.27 1.27)) (justify right bottom))
   )
@@
     (effects (font (size 1.27 1.27)) (justify right bottom))
   )
-  (label "D3_2" (at 195.58 152.4 180)
+  (label "D3_2" (at 195.58 269.24 180)
     (effects (font (size 1.27 1.27)) (justify right bottom))
   )
@@
     (effects (font (size 1.27 1.27)) (justify right bottom))
   )
-  (label "D3_7" (at 195.58 165.1 180)
+  (label "D3_7" (at 195.58 233.68 180)
     (effects (font (size 1.27 1.27)) (justify right bottom))
   )
@@
     (effects (font (size 1.27 1.27)) (justify left bottom))
   )
-  (label "D5_11" (at 195.58 231.14 180)
+  (label "D5_11" (at 195.58 149.86 180)
     (effects (font (size 1.27 1.27)) (justify right bottom))
   )
@@
     (effects (font (size 1.27 1.27)) (justify left bottom))
   )
-  (label "D3_5" (at 195.58 160.02 180)
+  (label "D3_5" (at 195.58 248.92 180)
     (effects (font (size 1.27 1.27)) (justify right bottom))
   )
@@
     (effects (font (size 1.27 1.27)) (justify right bottom))
   )
-  (label "D4_3" (at 195.58 246.38 180)
+  (label "D4_3" (at 195.58 185.42 180)
     (effects (font (size 1.27 1.27)) (justify right bottom))
   )
@@
     (effects (font (size 1.27 1.27)) (justify right bottom))
   )
-  (label "D4_5" (at 195.58 251.46 180)
+  (label "D4_5" (at 195.58 162.56 180)
     (effects (font (size 1.27 1.27)) (justify right bottom))
   )
@@
     (effects (font (size 1.27 1.27)) (justify left bottom))
   )
-  (label "D4_12" (at 195.58 269.24 180)
+  (label "D4_12" (at 195.58 243.84 180)
     (effects (font (size 1.27 1.27)) (justify right bottom))
   )
@@
     (effects (font (size 1.27 1.27)) (justify left bottom))
   )
-  (label "D4_8" (at 195.58 259.08 180)
+  (label "D4_8" (at 195.58 157.48 180)
     (effects (font (size 1.27 1.27)) (justify right bottom))
   )
@@
     (effects (font (size 1.27 1.27)) (justify left bottom))
   )
-  (label "ADC2_OE_N" (at 63.5 177.8 180)
+  (label "ADC2_OE_N" (at 195.58 228.6 180)
     (effects (font (size 1.27 1.27)) (justify right bottom))
   )
@@
     (effects (font (size 1.27 1.27)) (justify right bottom))
   )
-  (label "D3_8" (at 195.58 167.64 180)
+  (label "D3_8" (at 195.58 231.14 180)
     (effects (font (size 1.27 1.27)) (justify right bottom))
   )
@@
     (effects (font (size 1.27 1.27)) (justify right bottom))
   )
-  (label "D5_3" (at 195.58 190.5 180)
+  (label "D5_3" (at 195.58 180.34 180)
     (effects (font (size 1.27 1.27)) (justify right bottom))
   )
@@
     (effects (font (size 1.27 1.27)) (justify right bottom))
   )
-  (label "D5_4" (at 195.58 193.04 180)
+  (label "D5_4" (at 195.58 271.78 180)
     (effects (font (size 1.27 1.27)) (justify right bottom))
   )
@@
     (effects (font (size 1.27 1.27)) (justify left bottom))
   )
-  (label "D4_13" (at 195.58 271.78 180)
+  (label "D4_13" (at 195.58 266.7 180)
     (effects (font (size 1.27 1.27)) (justify right bottom))
   )
@@
     (effects (font (size 1.27 1.27)) (justify right bottom))
   )
-  (label "D3_11" (at 195.58 175.26 180)
+  (label "D3_11" (at 195.58 195.58 180)
     (effects (font (size 1.27 1.27)) (justify right bottom))
   )
@@
     (effects (font (size 1.27 1.27)) (justify right bottom))
   )
-  (label "D3_9" (at 195.58 170.18 180)
-    (effects (font (size 1.27 1.27)) (justify right bottom))
-  )
-  (label "D4_4" (at 195.58 248.92 180)
+  (label "D3_9" (at 195.58 220.98 180)
+    (effects (font (size 1.27 1.27)) (justify right bottom))
+  )
+  (label "D4_4" (at 195.58 167.64 180)
     (effects (font (size 1.27 1.27)) (justify right bottom))
   )
@@
     (effects (font (size 1.27 1.27)) (justify left bottom))
   )
-  (label "D3_13" (at 195.58 180.34 180)
+  (label "D3_13" (at 195.58 190.5 180)
     (effects (font (size 1.27 1.27)) (justify right bottom))
   )
@@
     (effects (font (size 1.27 1.27)) (justify left bottom))
   )
-  (label "D4_10" (at 195.58 264.16 180)
+  (label "D4_10" (at 195.58 254 180)
     (effects (font (size 1.27 1.27)) (justify right bottom))
   )
@@
     (effects (font (size 1.27 1.27)) (justify right bottom))
   )
-  (label "D4_2" (at 195.58 243.84 180)
+  (label "D4_2" (at 195.58 187.96 180)
     (effects (font (size 1.27 1.27)) (justify right bottom))
   )
@@
     (effects (font (size 1.27 1.27)) (justify left bottom))
   )
-  (label "D5_2" (at 195.58 187.96 180)
-    (effects (font (size 1.27 1.27)) (justify right bottom))
-  )
-  (label "D3_1" (at 195.58 149.86 180)
+  (label "D5_2" (at 195.58 261.62 180)
+    (effects (font (size 1.27 1.27)) (justify right bottom))
+  )
+  (label "D3_1" (at 195.58 256.54 180)
     (effects (font (size 1.27 1.27)) (justify right bottom))
   )
@@
     (effects (font (size 1.27 1.27)) (justify left bottom))
   )
-  (label "D4_7" (at 195.58 256.54 180)
+  (label "D4_7" (at 195.58 160.02 180)
     (effects (font (size 1.27 1.27)) (justify right bottom))
   )
@@
     (effects (font (size 1.27 1.27)) (justify left bottom))
   )
-  (label "D4_1" (at 195.58 241.3 180)
+  (label "D4_1" (at 195.58 193.04 180)
     (effects (font (size 1.27 1.27)) (justify right bottom))
   )
@@
     (effects (font (size 1.27 1.27)) (justify right bottom))
   )
-  (label "D5_0" (at 195.58 182.88 180)
+  (label "D5_0" (at 195.58 213.36 180)
     (effects (font (size 1.27 1.27)) (justify right bottom))
   )
@@
     (effects (font (size 1.27 1.27)) (justify right bottom))
   )
-  (label "D3_3" (at 195.58 154.94 180)
-    (effects (font (size 1.27 1.27)) (justify right bottom))
-  )
-  (label "D3_6" (at 195.58 162.56 180)
+  (label "D3_3" (at 195.58 259.08 180)
+    (effects (font (size 1.27 1.27)) (justify right bottom))
+  )
+  (label "D3_6" (at 195.58 246.38 180)
     (effects (font (size 1.27 1.27)) (justify right bottom))
   )
@@
     (effects (font (size 1.27 1.27)) (justify left bottom))
   )
-  (label "D4_11" (at 195.58 266.7 180)
+  (label "D4_11" (at 195.58 241.3 180)
     (effects (font (size 1.27 1.27)) (justify right bottom))
   )
@@
     (effects (font (size 1.27 1.27)) (justify left bottom))
   )
-  (label "D4_0" (at 195.58 238.76 180)
+  (label "D4_0" (at 195.58 182.88 180)
     (effects (font (size 1.27 1.27)) (justify right bottom))
   )
@@
     (effects (font (size 1.27 1.27)) (justify right bottom))
   )
-  (label "D5_12" (at 195.58 233.68 180)
+  (label "D5_12" (at 195.58 147.32 180)
     (effects (font (size 1.27 1.27)) (justify right bottom))
   )
@@
     (effects (font (size 1.27 1.27)) (justify left bottom))
   )
-  (label "D3_4" (at 195.58 157.48 180)
+  (label "D3_4" (at 195.58 251.46 180)
     (effects (font (size 1.27 1.27)) (justify right bottom))
   )
@@
     (effects (font (size 1.27 1.27)) (justify right bottom))
   )
-  (label "D5_7" (at 195.58 220.98 180)
+  (label "D5_7" (at 195.58 170.18 180)
     (effects (font (size 1.27 1.27)) (justify right bottom))
   )
@@
     (effects (font (size 1.27 1.27)) (justify right bottom))
   )
-  (label "ADC2_CS_N" (at 195.58 213.36 180)
+  (label "ADC2_CS_N" (at 195.58 238.76 180)
     (effects (font (size 1.27 1.27)) (justify right bottom))
   )
@@
     (effects (font (size 1.27 1.27)) (justify left bottom))
   )
-  (label "D5_6" (at 195.58 198.12 180)
+  (label "D5_6" (at 195.58 177.8 180)
     (effects (font (size 1.27 1.27)) (justify right bottom))
   )
@@
     (effects (font (size 1.27 1.27)) (justify right bottom))
   )
-  (label "D5_10" (at 195.58 228.6 180)
+  (label "D5_10" (at 63.5 177.8 180)
     (effects (font (size 1.27 1.27)) (justify right bottom))
   )
@@
     (effects (font (size 1.27 1.27)) (justify right bottom))
   )
-  (label "D5_8" (at 195.58 223.52 180)
+  (label "D5_8" (at 195.58 172.72 180)
     (effects (font (size 1.27 1.27)) (justify right bottom))
   )
@@
     (effects (font (size 1.27 1.27)) (justify right bottom))
   )
-  (label "D3_12" (at 195.58 177.8 180)
+  (label "D3_12" (at 195.58 198.12 180)
     (effects (font (size 1.27 1.27)) (justify right bottom))
   )
@@
     (effects (font (size 1.27 1.27)) (justify left bottom))
   )
-  (label "D3_0" (at 195.58 147.32 180)
+  (label "D3_0" (at 195.58 264.16 180)
     (effects (font (size 1.27 1.27)) (justify right bottom))
   )
@@
     (effects (font (size 1.27 1.27)) (justify right bottom))
   )
-  (label "D5_5" (at 195.58 195.58 180)
+  (label "D5_5" (at 195.58 175.26 180)
     (effects (font (size 1.27 1.27)) (justify right bottom))
   )
@@
     (effects (font (size 1.27 1.27)) (justify left bottom))
   )
-  (label "D4_6" (at 195.58 254 180)
-    (effects (font (size 1.27 1.27)) (justify right bottom))
-  )
+  (label "D4_6" (at 195.58 165.1 180)
+    (effects (font (size 1.27 1.27)) (justify right bottom))
+  )

Commit message: Continued layout of clocking subsystem, second ADC, and BGA fanout
Connections:
- net D5_13: now also U2.D3 (IO_L11N_T1_SRCC_35); no longer U2.H5 (IO_L18P_T2_35)
- net PLL_UWIRE_LE: now also U2.H5 (IO_L18P_T2_35); no longer U2.D3 (IO_L11N_T1_SRCC_35)
Changed lines of the file:
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@@
     (effects (font (size 1.27 1.27)) (justify right bottom))
   )
-  (label "D5_13" (at 195.58 236.22 180)
+  (label "D5_13" (at 195.58 203.2 180)
     (effects (font (size 1.27 1.27)) (justify right bottom))
   )
@@
     (effects (font (size 1.27 1.27)) (justify right))
   )
-  (hierarchical_label "PLL_UWIRE_LE" (shape output) (at 195.58 203.2 180)
+  (hierarchical_label "PLL_UWIRE_LE" (shape output) (at 195.58 236.22 180)
     (effects (font (size 1.27 1.27)) (justify right))
   )

Commit message: Hooked up power and analog connections to third ADC, no data bus yet
Connections:
- net D5_2: now also U2.C12 (IO_L11N_T1_SRCC_15); no longer U2.L3 (IO_L23P_T3_35)
- net D5_4: now also U2.C13 (IO_L12N_T1_MRCC_15); no longer U2.K5 (IO_25_35)
- net PLL_UWIRE_CLK: now also U2.K5 (IO_25_35); no longer U2.C12 (IO_L11N_T1_SRCC_15)
- net PLL_UWIRE_DATA: now also U2.L3 (IO_L23P_T3_35); no longer U2.C13 (IO_L12N_T1_MRCC_15)
Changed lines of the file:
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@@
   (title_block
     (title "Digitizer board")
-    (date "2023-02-01")
+    (date "2023-02-03")
     (rev "0.1")
     (company "A. Zonenberg")
@@
     (effects (font (size 1.27 1.27)) (justify right bottom))
   )
-  (label "D5_4" (at 195.58 271.78 180)
+  (label "D5_4" (at 130.81 208.28 180)
     (effects (font (size 1.27 1.27)) (justify right bottom))
   )
@@
     (effects (font (size 1.27 1.27)) (justify left bottom))
   )
-  (label "D5_2" (at 195.58 261.62 180)
+  (label "D5_2" (at 130.81 203.2 180)
     (effects (font (size 1.27 1.27)) (justify right bottom))
   )
@@
     (effects (font (size 1.27 1.27)) (justify right))
   )
-  (hierarchical_label "PLL_UWIRE_CLK" (shape output) (at 130.81 203.2 180)
+  (hierarchical_label "PLL_UWIRE_CLK" (shape output) (at 195.58 271.78 180)
     (effects (font (size 1.27 1.27)) (justify right))
   )
@@
     (effects (font (size 1.27 1.27)) (justify right))
   )
-  (hierarchical_label "PLL_UWIRE_DATA" (shape output) (at 130.81 208.28 180)
-    (effects (font (size 1.27 1.27)) (justify right))
-  )
+  (hierarchical_label "PLL_UWIRE_DATA" (shape output) (at 195.58 261.62 180)
+    (effects (font (size 1.27 1.27)) (justify right))
+  )
